File: main.kicad_sch (KiCad schematic)
At the start: 51 parts, among them J1 USB_C_Receptacle_USB2.0_16P, J2 Conn_ARM_JTAG_SWD_10, J4 UART, Q1 DMG1023UV-7, Q2 DMG1023UV-7, U1 STM32F411CEUx, U3 USBLC6-2SC6, U4 74LVC2T45DC, U5 74LVC2T45DC, U6 74LVC2T45DC, U7 74LVC2T45DC, U8 SPX3819M5-L-3-3, Y1 25 MHz 9pF

Commit message: schematic: initial design with stm32f103
Parts:
- removed C10: 1u, symbol Device:C
- removed C11, C12: 12p, symbol Device:C
- removed C13, C6, C7, C8, C9: 100n, symbol Device:C
- removed C23, C24: 4.7u, symbol Device:C_Polarized
- removed C4: 4.7u, symbol Device:C
- removed J2: Conn_ARM_JTAG_SWD_10, symbol Connector:Conn_ARM_JTAG_SWD_10
- removed L1: 10u, symbol Device:L
- removed Q2: DMG1023UV-7, footprints:SOTFL50P162X60-6N, symbol DMG1023UV-7:DMG1023UV-7
- removed RN1: 100, Resistor_THT:R_Array_SIP5, symbol Device:R_Network06_Split
- removed RN2: 330, Resistor_THT:R_Array_SIP5, symbol Device:R_Network04_Split
- removed TP1: ~{RESET}, symbol Connector:TestPoint
- removed U1: STM32F411CEUx, Package_DFN_QFN:QFN-48-1EP_7x7mm_P0.5mm_EP5.6x5.6mm, symbol MCU_ST_STM32F4:STM32F411CEUx
- removed Y1: 25 MHz 9pF, symbol Device:Crystal
- added C1, C2: 100n, Capacitor_SMD:C_0402_1005Metric, symbol Device:C
- added J2: Conn_ST_STDC14, Connector_PinHeader_1.27mm:PinHeader_2x07_P1.27mm_Vertical_SMD, symbol Connector:Conn_ST_STDC14
- added J3: DEBUG, Connector_PinHeader_1.27mm:PinHeader_1x05_P1.27mm_Horizontal, symbol Connector:Conn_01x05_Pin
- added unit 2 of Q1
- added Q2: DMG1024UV-7, footprints:SOTFL50P162X60-6N, symbol DMG1024UV-7:DMG1024UV-7
- added R1: 4.7k, Capacitor_SMD:C_0402_1005Metric, symbol Device:R
- added R10, R11: 330, Capacitor_SMD:C_0402_1005Metric, symbol Device:R
- added R12, R13, R14, R15, R19: 100, Capacitor_SMD:C_0402_1005Metric, symbol Device:R
- added R2, R3, R6: 10k, Capacitor_SMD:C_0402_1005Metric, symbol Device:R
- added SW1: DFU, Button_Switch_SMD:SW_Tactile_SPST_NO_Straight_CK_PTS636Sx25SMTRLFS, symbol Switch:SW_Push
- C10: renamed from C20; footprint (none) -> Capacitor_SMD:C_0402_1005Metric
- C11: renamed from C21; footprint (none) -> Capacitor_SMD:C_0402_1005Metric
- C12: renamed from C18; footprint (none) -> Capacitor_SMD:C_0402_1005Metric
- C13: renamed from C19; footprint (none) -> Capacitor_SMD:C_0402_1005Metric
- C3, R16, R17: footprint (none) -> Capacitor_SMD:C_0402_1005Metric
- C4: renamed from C22; footprint (none) -> Capacitor_SMD:C_0402_1005Metric
- C5: value 100n -> 4.7u; footprint (none) -> Capacitor_SMD:C_0402_1005Metric
- C6: renamed from C16; footprint (none) -> Capacitor_SMD:C_0402_1005Metric
- C7: renamed from C17; footprint (none) -> Capacitor_SMD:C_0402_1005Metric
- C8: renamed from C14; footprint (none) -> Capacitor_SMD:C_0402_1005Metric
- C9: renamed from C15; footprint (none) -> Capacitor_SMD:C_0402_1005Metric
- D1, D2, D3, D4: footprint (none) -> LED_SMD:LED_0805_2012Metric
- J1: footprint (none) -> Connector_USB:USB_C_Receptacle_Palconn_UTC16-G
- Q1: Height 0.6 -> (none); Manufacturer_Name Diodes Incorporated -> (none); Manufacturer_Part_Number DMG1023UV-7 -> (none); Mouser Part Number 621-DMG1023UV-7 -> (none); Mouser Price/Stock https://www.mouser.co.uk/ProductDetail/Diodes-Incorporated/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 -> (none)
- R18: value 10k -> 100; footprint (none) -> Capacitor_SMD:C_0402_1005Metric
- R4: renamed from R2; footprint (none) -> Capacitor_SMD:C_0402_1005Metric
- R5: renamed from R3; footprint (none) -> Capacitor_SMD:C_0402_1005Metric
- R7: value 22 -> 10k; footprint (none) -> Capacitor_SMD:C_0402_1005Metric
- R8: value 22 -> 330; footprint (none) -> Capacitor_SMD:C_0402_1005Metric
- R9: value 10k -> 330; footprint (none) -> Capacitor_SMD:C_0402_1005Metric
- renumbered U3 to U1, U8 to U2, U5 to U3, U7 to U5
Connections:
- net UART_RX is gone; now on net RX: U3.3 (2A)
- net UART_TX is gone; now on net TX: U5.2 (1A)
- net VBUS is gone; now on net +5V: J1.A4 (VBUS), J1.A9 (VBUS), J1.B4 (VBUS), J1.B9 (VBUS), U1.5 (VBUS), U2.1 (IN), U2.3 (EN)
- net GND: now also R8.2, R9.2, C1.2, C2.1, J2.11 (GNDDetect), J2.5 (GND), J2.7 (GND), J3.4 (Pin_4), Q2.1 (S), Q2.4 (S), R10.2, R11.2, R2.2, SW1.1; no longer D1.1 (K), D2.1 (K), D3.1 (K), D4.1 (K)
- net RX: now also R18.2, J2.13 (VCP_RX); no longer R17.2
- net TX: now also J2.14 (VCP_TX), R19.2; no longer R16.2
- net USB_D+: no longer R7.2
- net USB_D-: no longer R8.2
- net xRX: now also R19.1; no longer R17.1
- net xTCK: now also R14.1
- net xTDI: now also R17.1
- net xTDO: now also R16.1
- net xTMS: now also R15.1
- net xTX: now also R18.1; no longer R16.1
- net x~{RST}: now also R7.2, Q2.5 (G), Q2.6 (D), R13.1
- net STM32F103 MCU/ERROR_LED: now reaches D3.2 (A)
- net TVREF: now reaches R7.1
- net TVREF: now also J4.1 (Pin_1), J2.3 (VCC), Q1.3 (D), R1.1, R12.2
- net STM32F103 MCU/UART_LED: now reaches D2.2 (A)
- net +5V: now reaches C3.1
- net +3.3V: now reaches C5.1
- net +3.3V: now also C10.1, C12.1, C6.1, C8.1, D1.2 (A), Q1.6 (D), U2.5 (OUT), U3.1 (VCCA), U4.1 (VCCA), U4.5 (DIR), U5.1 (VCCA), U5.5 (DIR), U6.1 (VCCA), R3.1
- net STM32F103 MCU/IDLE/RUN_LED: now reaches D4.2 (A)
- net at R8.1: now also D1.1 (K)
- removed net 3.3V: C10.1, C12.1, C6.1, C8.1, Q1.3 (D1), U2.5 (OUT), U3.1 (VCCA), U4.1 (VCCA), U4.5 (DIR), U5.1 (VCCA), U5.5 (DIR), U6.1 (VCCA)
- net D+: no longer names the net of J1.A6 (D+), J1.B6 (D+), U1.3 (I/O2)
- net D-: no longer names the net of J1.A7 (D-), J1.B7 (D-), U1.1 (I/O1)
- removed net PWR_BR: Q1.2 (G2), Q1.5 (G1), R18.2, R9.2
- net TCK/SWCLK renamed TCK
- net TDO/TRACESWO renamed TDO
- net TMS/SWDIO renamed TMS
- removed net TPWR: J4.1 (Pin_1), Q1.6 (D2)
- net xTPWR renamed xVREF
- net xVREF: now also R12.1
- new net: J2.12 (~{RST}), R13.2
- new net: D2.1 (K), R9.1
- new net: J2.10 (JTDI/NC), R17.2
- new net: Q1.1 (S), Q1.4 (S), R6.1
- new net: D4.1 (K), R11.1
- new net: D3.1 (K), R10.1
- new net: J2.8 (JTDO/SWO), R16.2
- new net: J2.6 (JCLK/SWCLK), R14.2
- new net: J2.4 (JTMS/SWDIO), R15.2
- new net STM32F103 MCU/TRST: Q2.2 (G)
- new net STM32F103 MCU/TVREF: C1.1, R1.2, R2.1
- new net STM32F103 MCU/~{FORCE_DFU}: R3.2, SW1.2
- new net SWCLK: J3.3 (Pin_3)
- new net SWDIO: J3.5 (Pin_5)
- new net SWO: J3.2 (Pin_2)
- new net TRST_SENSE: Q2.3 (D)
- new net ~{ASSERT_TVREF}: Q1.2 (G), Q1.5 (G), R6.2
- new net ~{RESET}: C2.2, J3.1 (Pin_1)
- no-connect marks 20 -> 3
Other:
- added sheet STM32F103 MCU (stm32f103-mcu.kicad_sch)
- note added: "All unused I/Os must be tied to GND. (Section 8.1, Datasheet)"
- note added: "DIR = GND: <- DIR = VCC: ->"
- note added: "Debug Connectors"
- note added: "JTAG and SWD pins are multiplexed according to the connector everywhere but JTAG alone is used to label nets for brevity. Nets prefixed with either "T"(target device) or "x" (??)."
- note added: "Level Shifters"
- note added: "Microcontroller"
- note added: "Place ${/f1fc6258-4499-4f1b-936c-09bde8d994b8/3a76b143-a864-4074-abff-d5ea8ba2a739:REFERENCE} close to ${/f1fc6258-4499-4f1b-936c-09bde8d994b8/907ca9d1-e01e-4a83-a719-4f392d685990:REFERENCE} and keep VCC and GND traces short."
- note added: "Request 5V@0.5A."
- note added: "Series termination resistors to dampen ringing. STDC14 is a superset of the 10-pin ARM JTAG/SWD connector and only STDC14 has UART. The following conigurations are possible: - Unified: STDC14 on ${/f1fc6258-4499-4f1b-936c-09bde8d994b8/c7963dce-d9ad-4869-a1d6-a9894ba76f4f:REFERENCE} (Debug + UART), do not populate ${/f1fc6258-4499-4f1b-936c-09bde8d994b8/9a528976-fea6-40da-88a5-3aeb6df08928:REFEREN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"
- note added: "Supported target I/O voltage (TVREF) range is 1.7 V - 5 V. This info is used to scale down TVREF. TRST_SENSE must be internally pulled up in the firmware."
- note added: "TVREF Supply Control"
- note added: "USB-C Connector"
- note added: "Voltage Regulator"
- moved on the sheet: C10, C11, C12, C13, C4, C6, C7, C8, C9, D1, D2, D3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

Commit message: layout: initial design with added LCSC part metadata
Parts:
- C1, C10, C11, C12, C13, C2, C6, C7, C8, C9: LCSC Part (none) -> C60474
- C3, C5: LCSC Part (none) -> C23733
- C4: LCSC Part (none) -> C14663
- D1: footprint LED_SMD:LED_0805_2012Metric -> LED_SMD:LED_0402_1005Metric; LCSC Part (none) -> C2980183
- D2: footprint LED_SMD:LED_0805_2012Metric -> LED_SMD:LED_0402_1005Metric; LCSC Part (none) -> C779448
- D3: footprint LED_SMD:LED_0805_2012Metric -> LED_SMD:LED_0402_1005Metric; LCSC Part (none) -> C136765
- D4: footprint LED_SMD:LED_0805_2012Metric -> LED_SMD:LED_0402_1005Metric; LCSC Part (none) -> C20608782
- J1: footprint Connector_USB:USB_C_Receptacle_Palconn_UTC16-G -> Connector_USB:USB_C_Receptacle_GCT_USB4105-xx-A_16P_TopMnt_Horizontal; LCSC Part (none) -> C2988369
- J2: footprint Connector_PinHeader_1.27mm:PinHeader_2x07_P1.27mm_Vertical_SMD -> footprints:SAMTEC_FTSH-107-01-L-DV-K; LCSC Part (none) -> C46971079
- J3: footprint Connector_PinHeader_1.27mm:PinHeader_1x05_P1.27mm_Horizontal -> Connector_PinHeader_1.27mm:PinHeader_1x05_P1.27mm_Vertical; now not fitted
- J4: footprint Connector_PinHeader_1.27mm:PinHeader_1x04_P1.27mm_Horizontal -> Connector_PinHeader_1.27mm:PinHeader_1x04_P1.27mm_Vertical; now not fitted
- Q1: LCSC Part (none) -> C212298
- Q2: LCSC Part (none) -> C2759893
- R1: footprint Capacitor_SMD:C_0402_1005Metric -> Resistor_SMD:R_0402_1005Metric; LCSC Part (none) -> C105871
- R10, R11, R8, R9: footprint Capacitor_SMD:C_0402_1005Metric -> Resistor_SMD:R_0402_1005Metric; LCSC Part (none) -> C105875
- R12, R13, R14, R15, R16, R17, R18, R19: footprint Capacitor_SMD:C_0402_1005Metric -> Resistor_SMD:R_0402_1005Metric; LCSC Part (none) -> C106232
- R2, R3, R6, R7: footprint Capacitor_SMD:C_0402_1005Metric -> Resistor_SMD:R_0402_1005Metric; LCSC Part (none) -> C60490
- R4, R5: footprint Capacitor_SMD:C_0402_1005Metric -> Resistor_SMD:R_0402_1005Metric; LCSC Part (none) -> C25905
- SW1: footprint Button_Switch_SMD:SW_Tactile_SPST_NO_Straight_CK_PTS636Sx25SMTRLFS -> Button_Switch_SMD:SW_Push_SPST_NO_Alps_SKRK; LCSC Part (none) -> C720477
- U1: LCSC Part (none) -> C7519
- U2: LCSC Part (none) -> C9055
- U3, U4, U5, U6: LCSC Part (none) -> C15741
Connections:
- net +3.3V: now also R8.1; no longer D1.2 (A)
- net GND: now also D1.1 (K), D2.1 (K), D3.1 (K), D4.1 (K); no longer R10.2, R11.2, R8.2, R9.2
- net RX: no longer J2.13 (VCP_RX), J4.3 (Pin_3), R18.2
- net STM32F103 MCU/ERROR_LED: now also R10.1; no longer D3.2 (A)
- net STM32F103 MCU/IDLE/RUN_LED: now also R11.1; no longer D4.2 (A)
- net STM32F103 MCU/UART_LED: now also R9.1; no longer D2.2 (A)
- net TX: no longer J2.14 (VCP_TX), J4.2 (Pin_2), R19.2
- net xRX: now also R18.1; no longer R19.1
- net xTX: now also R19.1; no longer R18.1
- net D-: now reaches J1.A7 (D-), J1.B7 (D-), U1.1 (I/O1)
- net D+: now reaches J1.A6 (D+), J1.B6 (D+), U1.3 (I/O2)
- new net: D1.2 (A), R8.2
- new net: D2.2 (A), R9.2
- new net: D4.2 (A), R11.2
- new net: D3.2 (A), R10.2
- new net cRX: J2.13 (VCP_RX), J4.3 (Pin_3), R18.2
- new net cTX: J2.14 (VCP_TX), J4.2 (Pin_2), R19.2
Other:
- note added: "JTAG and SWD pins are multiplexed according to the connector everywhere but JTAG alone is used to label nets for brevity. Nets are prefixed with either "T"(target device) or "x" (post series termination)."
- note added: "Series termination resistors to dampen ringing. STDC14 is a superset of the 10-pin ARM JTAG/SWD connector and only STDC14 has UART. The following conigurations are possible [with Samtec connector]: - STDC14 on ${/f1fc6258-4499-4f1b-936c-09bde8d994b8/c7963dce-d9ad-4869-a1d6-a9894ba76f4f:REFERENCE} (Debug + UART) [FTSH-107-01-L-DV-K] - 10-pin ARM JTAG/SWD on ${/f1fc6258-4499-4f1b-936c-09bde8d994b8/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"
- note removed: "JTAG and SWD pins are multiplexed according to the connector everywhere but JTAG alone is used to label nets for brevity. Nets prefixed with either "T"(target device) or "x" (??)."
- note removed: "Series termination resistors to dampen ringing. STDC14 is a superset of the 10-pin ARM JTAG/SWD connector and only STDC14 has UART. The following conigurations are possible: - Unified: STDC14 on ${/f1fc6258-4499-4f1b-936c-09bde8d994b8/c7963dce-d9ad-4869-a1d6-a9894ba76f4f:REFERENCE} (Debug + UART), do not populate ${/f1fc6258-4499-4f1b-936c-09bde8d994b8/9a528976-fea6-40da-88a5-3aeb6df08928:REFEREN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"
- title: Black Magic Probe -> μProbe
- moved on the sheet: D1, D2, D3, D4, R10, R11, R18, R19, R8, R9

Commit message: schematic: fix C4 LCSC part number and STM32F1 component variant
The BMP firmware cannot be flashed onto the STM32F103C8Tx (64 KiB
variant) due to size constraints. The STM32F103CBUx was used in the
reference schematic but somehow got overlooked during the design.
Parts:
- C4: LCSC Part C14663 -> C15195
- J3, J4: now left out of the parts list
Changed lines of the file:
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@@
 			)
 		)
-		(property "LCSC Part" "C14663"
+		(property "LCSC Part" "C15195"
 			(at 111.76 33.02 0)
 			(effects
@@
 		(unit 1)
 		(exclude_from_sim no)
-		(in_bom yes)
+		(in_bom no)
 		(on_board yes)
 		(dnp yes)
@@
 		(unit 1)
 		(exclude_from_sim no)
-		(in_bom yes)
+		(in_bom no)
 		(on_board yes)
 		(dnp yes)
