File: main.kicad_pcb (KiCad board)
At the start: 2 copper layers, 18 x 36 mm, 62 parts, among them J1 USB_C_Receptacle_USB2.0_16P, J2 Conn_ST_STDC14, J3 DEBUG, J4 UART, Q1 DMG1023UV-7, Q2 DMG1024UV-7, SW1 DFU, U1 USBLC6-2SC6, U2 SPX3819M5-L-3-3, U3 74LVC2T45DC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

Commit message: schematic: fix LCSC part number for STM32F1 MCU
Parts:
- U7: value STM32F103CBUx -> STM32F103CBTx
Changed lines of the file:
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@@
 			)
 		)
-		(property "Value" "STM32F103CBUx"
+		(property "Value" "STM32F103CBTx"
 			(at 0 5.85 90)
 			(layer "F.Fab")
@@
 			)
 		)
-		(property "LCSC Part" "C8734"
+		(property "LCSC Part" "C8304"
 			(at 0 0 90)
 			(unlocked yes)
